File: RP2040_board/RP2040_devBoard.kicad_pcb (KiCad board)
At the start: 2 copper layers, 26 x 56.9 mm, 85 parts, among them J1 USB_B_Micro, J2 Conn_01x20_Male, J3 Conn_01x20_Male, J4 Conn_01x03_Male, SW1 SW_Push, U1 RP2040, U2 AMS1117, U3 W25Q128JVS, Y1 Crystal

Commit message: board finish
Parts:
- removed kibuzzard-648F360B: G***, kibuzzard-648F360B
- removed kibuzzard-648F3618: G***, kibuzzard-648F3618
- removed kibuzzard-648F362B: G***, kibuzzard-648F362B
- removed kibuzzard-648F3636: G***, kibuzzard-648F3636
- removed kibuzzard-648F363F: G***, kibuzzard-648F363F
- removed kibuzzard-648F364A: G***, kibuzzard-648F364A
- removed the kibuzzard-648F3652 at (60.7, 62.0)
- removed kibuzzard-648F365C: G***, kibuzzard-648F365C
- removed kibuzzard-648F3665: G***, kibuzzard-648F3665
- removed kibuzzard-648F366D: G***, kibuzzard-648F366D
- removed kibuzzard-648F3677: G***, kibuzzard-648F3677
- removed kibuzzard-648F3868: G***, kibuzzard-648F3868
- added kibuzzard-64910299: G***, kibuzzard-64910299, B.Cu at (60.6, 46.8)
- added kibuzzard-6491029F: G***, kibuzzard-6491029F, B.Cu at (60.5, 49.4)
- added kibuzzard-649102A3: G***, kibuzzard-649102A3, B.Cu at (60.6, 51.8)
- added kibuzzard-649102AA: G***, kibuzzard-649102AA, B.Cu at (60.6, 54.4)
- added kibuzzard-649102B0: G***, kibuzzard-649102B0, B.Cu at (60.6, 56.9)
- added kibuzzard-649102B6: G***, kibuzzard-649102B6, B.Cu at (60.6, 59.5)
- added kibuzzard-649102CC: G***, kibuzzard-649102CC, B.Cu at (60.5, 64.6)
- added kibuzzard-649102D1: G***, kibuzzard-649102D1, B.Cu at (60.5, 67.1)
- added kibuzzard-649102D9: G***, kibuzzard-649102D9, B.Cu at (60.6, 69.6)
- added kibuzzard-649102E1: G***, kibuzzard-649102E1, B.Cu at (60.5, 72.2)
- added kibuzzard-64910390: G***, kibuzzard-64910390, B.Cu at (60.6, 62.0)
- added kibuzzard-649125AB: G***, kibuzzard-649125AB, B.Cu at (68.8, 92.9)
- D1, D3: footprint LED_SMD:LED_1206_3216Metric -> LED_SMD:LED_0603_1608Metric
- SW1: value SW_Push -> PTS815_SJM_250_SMTR_LFS; footprint Tactile_SW:SW_PTS636_SMT-G_5_CNK -> FOOTPRINTS_s1:SW4_PTS815 SJM 250 SMTR LFS_CNK
- Y1: footprint Crystal:Crystal_SMD_HC49-SD -> MCU_RaspberryPi_and_Boards:Crystal_SMD_HC49-US
- moved G*** 3.31 mm to (68.9, 49.3)
- moved G*** 2.72 mm to (68.8, 53.4)
- moved G*** 0.93 mm to (62.4, 79.0)
- moved SW1 0.92 mm to (62.8, 51.1)
- moved G*** 0.82 mm to (62.4, 83.0)
- moved R6 0.82 mm to (74.3, 46.8), turned to -90 degrees
- moved C12 0.67 mm to (74.2, 62.3)
- moved D1 0.58 mm to (74.3, 50.6)
- moved C14 0.55 mm to (66.4, 56.0)
Connections:
- SW1 pad 2: /USB_BOOT -> (no net)
Routing:
- net GND: track 101.9 -> 109.8 mm, vias 45 -> 43
- net /GPIO0: track 37.9 -> 36.6 mm
- net /GPIO15: track 20.9 -> 20.2 mm
- net /GPIO8: track 13.6 -> 12.9 mm
- net /USB_BOOT: track 3.24 -> 2.63 mm
- net VBUS: track 24.0 -> 24.6 mm
- net Net-(D3-Pad1): track 5.19 -> 4.69 mm

Commit message: added the rest of files for the repo
Parts:
- removed the G*** at (68.9, 49.3)
- removed the G*** at (68.8, 53.4)
- added G***: LOGO, LOGO, B.Cu at (68.8, 60.1)
- added G***: LOGO, LOGO, B.Cu at (68.9, 53.7)
- moved C14 1.20 mm to (65.4, 56.7), turned to 180 degrees
- moved C13 0.43 mm to (72.3, 50.0)
